File: binary_interfacer_kicad/binary_interfacer_kicad.kicad_sch (KiCad schematic)
At the start: 21 parts, among them J1 Conn_01x16_Male, J2 Conn_01x04_Male, U1 74HC165, U2 74HC165

Commit message: Third Deliverable
Added a keypad and binary outputs to the device. So a number can be
entered on the keypad, and outputted as binary on the bus.
Parts:
- added SW1, SW10, SW2, SW3, SW4, SW5, SW6, SW7, SW8, SW9: SW_SPST, symbol Switch:SW_SPST
- added SW11: SW_SPDT, symbol Switch:SW_SPDT
- added U3, U4: 74HC595, symbol 74xx:74HC595
Connections:
- net +5V: now also SW11.3 (C), U3.10 (~{SRCLR}), U3.16 (VCC), U4.10 (~{SRCLR}), U4.16 (VCC)
- net BIT0: now also U3.15 (QA)
- net BIT1: now also U3.1 (QB)
- net BIT10: now also U4.2 (QC)
- net BIT11: now also U4.3 (QD)
- net BIT12: now also U4.4 (QE)
- net BIT13: now also U4.5 (QF)
- net BIT14: now also U4.6 (QG)
- net BIT15: now also U4.7 (QH)
- net BIT2: now also U3.2 (QC)
- net BIT3: now also U3.3 (QD)
- net BIT4: now also U3.4 (QE)
- net BIT5: now also U3.5 (QF)
- net BIT6: now also U3.6 (QG)
- net BIT7: now also U3.7 (QH)
- net BIT8: now also U4.15 (QA)
- net BIT9: now also U4.1 (QB)
- net CLK: now also U3.11 (SRCLK), U4.11 (SRCLK)
- net DATA: now also U3.14 (SER)
- net GND: now also SW1.2 (B), SW10.2 (B), SW11.1 (A), SW2.2 (B), SW3.2 (B), SW4.2 (B), SW5.2 (B), SW6.2 (B), SW7.2 (B), SW8.2 (B), SW9.2 (B), U3.8 (GND), U4.8 (GND)
- net LOAD: now also U3.12 (RCLK), U4.12 (RCLK)
- net KEY9: now reaches A1.10 (D7)
- net KEY9: now also SW3.1 (A)
- net KEY8: now reaches A1.11 (D8)
- net KEY8: now also SW2.1 (A)
- net KEY7: now reaches A1.12 (D9)
- net KEY7: now also SW1.1 (A)
- net KEY6: now reaches A1.13 (D10)
- net KEY6: now also SW6.1 (A)
- net KEY5: now reaches A1.15 (D12)
- net KEY5: now also SW5.1 (A)
- net KEY0: now reaches A1.19 (A0)
- net KEY0: now also SW10.1 (A)
- net KEY1: now reaches A1.20 (A1)
- net KEY1: now also SW7.1 (A)
- net KEY2: now reaches A1.21 (A2)
- net KEY2: now also SW8.1 (A)
- net KEY3: now reaches A1.22 (A3)
- net KEY3: now also SW9.1 (A)
- net MODE_SWITCH: now reaches A1.5 (D2)
- net MODE_SWITCH: now also SW11.2 (B), U3.13 (~{OE}), U4.13 (~{OE})
- net KEY4: now reaches A1.6 (D3)
- net KEY4: now also SW4.1 (A)
- new net: U3.9 (QH'), U4.14 (SER)
- no-connect marks 25 -> 15
Other:
- note added: "Bus Connectors"
- note added: "Bus I/O Connectors"
- note added: "Bus Input Shift Registers"
- note added: "Bus Output Shift Registers"
- note added: "Bus pulldowns - 10k"
- note added: "Mode Switch"
- note added: "Numpad"
- note removed: "Bus"
- note removed: "Bus Inputs"
- note removed: "Bus pulldowns"
- moved on the sheet: A1, J1, J2, R1, U1, U2

Commit message: Fourth deliverable
Changed mode select from a toggle switch to a push button
Parts:
- removed SW11: SW_SPDT, symbol Switch:SW_SPDT
- added SW12: SW_SPST, symbol Switch:SW_SPST
Connections:
- net GND: now also SW12.2 (B)
- net MODE_SWITCH: now also SW12.1 (A); no longer U3.13 (~{OE}), U4.13 (~{OE})
- net OUTPUT: now reaches A1.14 (D11)
- net OUTPUT: now also U3.13 (~{OE}), U4.13 (~{OE})
- no-connect marks 15 -> 14
Other:
- note removed: "Mode Switch"
Changed lines of the file:
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@@
   (no_connect (at 336.55 67.31))
   (no_connect (at 383.54 67.31))
-  (no_connect (at 123.19 187.96))
   (wire (pts (xy 287.02 146.05) (xy 287.02 147.32))
     (stroke (width 0) (type default))
@@
     (stroke (width 0) (type default))
   )
+  (wire (pts (xy 52.07 165.1) (xy 52.07 166.37))
+    (stroke (width 0) (type default))
+  )
   (wire (pts (xy 274.32 146.05) (xy 274.32 147.32))
     (stroke (width 0) (type default))
@@
     (stroke (width 0) (type default))
   )
-  (wire (pts (xy 74.93 76.2) (xy 73.66 76.2))
-    (stroke (width 0) (type default))
-  )
   (wire (pts (xy 41.91 135.89) (xy 41.91 137.16))
     (stroke (width 0) (type default))
@@
     (stroke (width 0) (type default))
   )
+  (wire (pts (xy 121.92 187.96) (xy 123.19 187.96))
+    (stroke (width 0) (type default))
+  )
   (wire (pts (xy 228.6 73.66) (xy 229.87 73.66))
     (stroke (width 0) (type default))
@@
     (stroke (width 0) (type default))
   )
-  (wire (pts (xy 73.66 74.93) (xy 73.66 76.2))
-    (stroke (width 0) (type default))
-  )
   (wire (pts (xy 309.88 69.85) (xy 311.15 69.85))
     (stroke (width 0) (type default))
@@
     (stroke (width 0) (type default))
   )
+  (wire (pts (xy 52.07 176.53) (xy 52.07 179.07))
+    (stroke (width 0) (type default))
+  )
   (wire (pts (xy 356.87 95.25) (xy 358.14 95.25))
     (stroke (width 0) (type default))
@@
     (stroke (width 0) (type default))
   )
-  (wire (pts (xy 73.66 82.55) (xy 73.66 81.28))
-    (stroke (width 0) (type default))
-  )
   (wire (pts (xy 261.62 146.05) (xy 261.62 147.32))
     (stroke (width 0) (type default))
@@
     (stroke (width 0) (type default))
   )
-  (wire (pts (xy 73.66 81.28) (xy 74.93 81.28))
-    (stroke (width 0) (type default))
-  )
   (wire (pts (xy 320.04 153.67) (xy 320.04 154.94))
     (stroke (width 0) (type default))
@@
     (stroke (width 0) (type default))
   )
-  (wire (pts (xy 85.09 78.74) (xy 86.36 78.74))
-    (stroke (width 0) (type default))
-  )
   (wire (pts (xy 297.18 153.67) (xy 297.18 154.94))
     (stroke (width 0) (type default))
@@
   (wire (pts (xy 121.92 170.18) (xy 123.19 170.18))
     (stroke (width 0) (type default))
-  )
-  (rectangle (start 68.58 67.31) (end 105.41 88.9)
-    (stroke (width 0) (type default))
-    (fill (type none))
   )
   (rectangle (start 102.87 135.89) (end 200.66 213.36)
@@
     (effects (font (size 3 3) (thickness 0.6) bold) (justify left bottom))
   )
-  (text "Mode Switch" (at 68.58 66.04 0)
-    (effects (font (size 3 3) (thickness 0.6) bold) (justify left bottom))
-  )
   (text "Numpad" (at 19.05 66.04 0)
     (effects (font (size 3 3) (thickness 0.6) bold) (justify left bottom))
@@
     )
   )
+  (global_label "MODE_SWITCH" (shape input) (at 52.07 165.1 90) (fields_autoplaced)
+    (effects (font (size 1.27 1.27)) (justify left))
+    (property "Intersheetrefs" "${INTERSHEET_REFS}" (at 52.07 149.1919 90)
+      (effects (font (size 1.27 1.27)) (justify left) hide)
+    )
+  )
   (global_label "BIT8" (shape input) (at 276.86 71.12 0) (fields_autoplaced)
     (effects (font (size 1.27 1.27)) (justify left))
@@
     )
   )
-  (global_label "MODE_SWITCH" (shape input) (at 254 87.63 270) (fields_autoplaced)
-    (effects (font (size 1.27 1.27)) (justify right))
-    (property "Intersheetrefs" "${INTERSHEET_REFS}" (at 254 103.5381 90)
-      (effects (font (size 1.27 1.27)) (justify right) hide)
-    )
-  )
   (global_label "CLK" (shape input) (at 205.74 76.2 180) (fields_autoplaced)
     (effects (font (size 1.27 1.27)) (justify right))
@@
     )
   )
+  (global_label "OUTPUT" (shape input) (at 121.92 187.96 180) (fields_autoplaced)
+    (effects (font (size 1.27 1.27)) (justify right))
+    (property "Intersheetrefs" "${INTERSHEET_REFS}" (at 111.8175 187.96 0)
+      (effects (font (size 1.27 1.27)) (justify right) hide)
+    )
+  )
   (global_label "KEY3" (shape input) (at 52.07 135.89 90) (fields_autoplaced)
     (effects (font (size 1.27 1.27)) (justify left))
@@
     )
   )
-  (global_label "MODE_SWITCH" (shape input) (at 86.36 78.74 0) (fields_autoplaced)
-    (effects (font (size 1.27 1.27)) (justify left))
-    (property "Intersheetrefs" "${INTERSHEET_REFS}" (at 102.2681 78.74 0)
-      (effects (font (size 1.27 1.27)) (justify left) hide)
-    )
-  )
-  (global_label "MODE_SWITCH" (shape input) (at 207.01 87.63 270) (fields_autoplaced)
-    (effects (font (size 1.27 1.27)) (justify right))
-    (property "Intersheetrefs" "${INTERSHEET_REFS}" (at 207.01 103.5381 90)
-      (effects (font (size 1.27 1.27)) (justify right) hide)
-    )
-  )
   (global_label "LOAD" (shape input) (at 356.87 90.17 180) (fields_autoplaced)
     (effects (font (size 1.27 1.27)) (justify right))
@@
     )
   )
+  (global_label "OUTPUT" (shape input) (at 207.01 87.63 270) (fields_autoplaced)
+    (effects (font (size 1.27 1.27)) (justify right))
+    (property "Intersheetrefs" "${INTERSHEET_REFS}" (at 207.01 97.7325 90)
+      (effects (font (size 1.27 1.27)) (justify right) hide)
+    )
+  )
   (global_label "KEY2" (shape input) (at 149.86 180.34 0) (fields_autoplaced)
     (effects (font (size 1.27 1.27)) (justify left))
@@
     )
   )
+  (global_label "OUTPUT" (shape input) (at 254 87.63 270) (fields_autoplaced)
+    (effects (font (size 1.27 1.27)) (justify right))
+    (property "Intersheetrefs" "${INTERSHEET_REFS}" (at 254 97.7325 90)
+      (effects (font (size 1.27 1.27)) (justify right) hide)
+    )
+  )
   (global_label "KEY5" (shape input) (at 41.91 106.68 90) (fields_autoplaced)
     (effects (font (size 1.27 1.27)) (justify left))
@@
     (property "Intersheetrefs" "${INTERSHEET_REFS}" (at 114.5994 170.18 0)
       (effects (font (size 1.27 1.27)) (justify right) hide)
+    )
+  )
+  (symbol (lib_id "Switch:SW_SPST") (at 52.07 171.45 270) (unit 1)
+    (in_bom yes) (on_board yes) (dnp no) (fields_autoplaced)
+    (property "Reference" "SW12" (at 54.61 171.45 90)
+      (effects (font (size 1.27 1.27)) (justify left))
+    )
+    (property "Value" "SW_SPST" (at 54.61 172.72 90)
+      (effects (font (size 1.27 1.27)) (justify left) hide)
+    )
+    (property "Footprint" "" (at 52.07 171.45 0)
+      (effects (font (size 1.27 1.27)) hide)
+    )
+    (property "Datasheet" "~" (at 52.07 171.45 0)
+      (effects (font (size 1.27 1.27)) hide)
+    )
+    (pin "1")
+    (pin "2")
+    (instances
+      (project "binary_interfacer_kicad"
+        (path "/c7089597-100c-4b8c-b94a-219051c81e2d"
+          (reference "SW12") (unit 1)
+        )
+      )
     )
   )
@@
     )
   )
-  (symbol (lib_id "Switch:SW_SPDT") (at 80.01 78.74 180) (unit 1)
-    (in_bom yes) (on_board yes) (dnp no) (fields_autoplaced)
-    (property "Reference" "SW11" (at 80.01 73.66 0)
-      (effects (font (size 1.27 1.27)))
-    )
-    (property "Value" "SW_SPDT" (at 80.01 73.66 0)
-      (effects (font (size 1.27 1.27)) hide)
-    )
-    (property "Footprint" "" (at 80.01 78.74 0)
-      (effects (font (size 1.27 1.27)) hide)
-    )
-    (property "Datasheet" "~" (at 80.01 78.74 0)
-      (effects (font (size 1.27 1.27)) hide)
-    )
-    (pin "1")
-    (pin "2")
-    (pin "3")
-    (instances
-      (project "binary_interfacer_kicad"
-        (path "/c7089597-100c-4b8c-b94a-219051c81e2d"
-          (reference "SW11") (unit 1)
-        )
-      )
-    )
-  )
   (symbol (lib_id "Device:R") (at 312.42 149.86 0) (unit 1)
     (in_bom yes) (on_board yes) (dnp no)
@@
     )
   )
-  (symbol (lib_name "GND_1") (lib_id "power:GND") (at 73.66 82.55 0) (unit 1)
-    (in_bom yes) (on_board yes) (dnp no) (fields_autoplaced)
-    (property "Reference" "#PWR018" (at 73.66 88.9 0)
-      (effects (font (size 1.27 1.27)) hide)
-    )
-    (property "Value" "GND" (at 73.66 87.63 0)
+  (symbol (lib_name "GND_1") (lib_id "power:GND") (at 52.07 179.07 0) (unit 1)
+    (in_bom yes) (on_board yes) (dnp no) (fields_autoplaced)
+    (property "Reference" "#PWR020" (at 52.07 185.42 0)
+      (effects (font (size 1.27 1.27)) hide)
+    )
+    (property "Value" "GND" (at 52.07 184.15 0)
       (effects (font (size 1.27 1.27)))
     )
-    (property "Footprint" "" (at 73.66 82.55 0)
-      (effects (font (size 1.27 1.27)) hide)
-    )
-    (property "Datasheet" "" (at 73.66 82.55 0)
-      (effects (font (size 1.27 1.27)) hide)
-    )
-    (pin "1")
-    (instances
-      (project "binary_interfacer_kicad"
-        (path "/c7089597-100c-4b8c-b94a-219051c81e2d"
-          (reference "#PWR018") (unit 1)
+    (property "Footprint" "" (at 52.07 179.07 0)
+      (effects (font (size 1.27 1.27)) hide)
+    )
+    (property "Datasheet" "" (at 52.07 179.07 0)
+      (effects (font (size 1.27 1.27)) hide)
+    )
+    (pin "1")
+    (instances
+      (project "binary_interfacer_kicad"
+        (path "/c7089597-100c-4b8c-b94a-219051c81e2d"
+          (reference "#PWR020") (unit 1)
         )
       )
@@
         )
       )
-    )
-  )
-  (symbol (lib_id "power:+5V") (at 73.66 74.93 0) (unit 1)
-    (in_bom yes) (on_board yes) (dnp no) (fields_autoplaced)
-    (property "Reference" "#PWR019" (at 73.66 78.74 0)
-      (effects (font (size 1.27 1.27)) hide)
-    )
-    (property "Value" "+5V" (at 73.66 69.85 0)
-      (effects (font (size 1.27 1.27)))
-    )
-    (property "Footprint" "" (at 73.66 74.93 0)
-      (effects (font (size 1.27 1.27)) hide)
-    )
-    (property "Datasheet" "" (at 73.66 74.93 0)
-      (effects (font (size 1.27 1.27)) hide)
-    )
-    (pin "1")
-    (instances
-      (project "binary_interfacer_kicad"
-        (path "/c7089597-100c-4b8c-b94a-219051c81e2d"
-          (reference "#PWR019") (unit 1)
-        )
-      )
